File: NRF52840.sch (KiCad schematic (older format))
At the start: 27 parts, among them J1 Conn_01x04, J2 USB_A, U1 nRF52840, Y1 32M

Commit message: ...
Parts:
- removed C10, C13, C25: NC, Capacitor_SMD:C_0402_1005Metric, symbol Device:C
- removed C12, C8: 100nF, Capacitor_SMD:C_0402_1005Metric, symbol Device:C
- removed C14: 1.0uF, Capacitor_SMD:C_0603_1608Metric, symbol Device:C
- removed C19, C6: 4.7uF, Capacitor_SMD:C_0603_1608Metric, symbol Device:C
- removed C26: 1.5pF, Capacitor_SMD:C_0402_1005Metric, symbol Device:C
- removed C7: 100nf, Capacitor_SMD:C_0402_1005Metric, symbol Device:C
- removed J1: Conn_01x04, zhangxiaofei:SWD, symbol Connector_Generic:Conn_01x04
- removed R1: 0R, Capacitor_SMD:C_0402_1005Metric, symbol Device:R
- added J1: Conn_01x02, zhangxiaofei:SWD_2_PIN, symbol Connector_Generic:Conn_01x02
Connections:
- wire segments 94 -> 62
- no-connect marks 51 -> 57

Commit message: ...
Parts:
- removed J1: Conn_01x02, zhangxiaofei:SWD_2_PIN, symbol Connector_Generic:Conn_01x02
- added C10, C13: NC, Capacitor_SMD:C_0201_0603Metric, symbol Device:C
- added C12, C7, C8: 100nF, Capacitor_SMD:C_0201_0603Metric, symbol Device:C
- added C14: 1.0uf, Capacitor_SMD:C_0402_1005Metric, symbol Device:C
- added C19, C6: 4.7uF, Capacitor_SMD:C_0402_1005Metric, symbol Device:C
- added J1: Conn_01x04, zhangxiaofei:SWD, symbol Connector_Generic:Conn_01x04
- C1, C11, C2, C5: footprint Capacitor_SMD:C_0402_1005Metric -> Capacitor_SMD:C_0201_0603Metric
- C15, C20: footprint Capacitor_SMD:C_0603_1608Metric -> Capacitor_SMD:C_0402_1005Metric
- C3: value 1.0pF -> 0.8pF; footprint Capacitor_SMD:C_0402_1005Metric -> Capacitor_SMD:C_0201_0603Metric
- C4: value 1.0pF -> 0.5pF; footprint Capacitor_SMD:C_0402_1005Metric -> Capacitor_SMD:C_0201_0603Metric
- J2: footprint zhangxiaofei:USB_PCB -> zhangxiaofei:mini_usb
- L1: value 3.9nH -> 4.7nH; footprint Inductor_SMD:L_0402_1005Metric -> Inductor_SMD:L_0201_0603Metric
- U1: symbol MCU_Nordic:nRF52840 -> NRF52840-rescue:nRF52840-MCU_Nordic
Connections:
- wire segments 62 -> 89
- no-connect marks 57 -> 51

Commit message: ...
Parts:
- removed C13: NC, Capacitor_SMD:C_0201_0603Metric, symbol Device:C
- removed C14: 1.0uf, Capacitor_SMD:C_0402_1005Metric, symbol Device:C
- removed C15: 1.0uF, Capacitor_SMD:C_0402_1005Metric, symbol Device:C
- removed C16: 4.7uF, Capacitor_SMD:C_0603_1608Metric, symbol Device:C
- removed C19, C20: 4.7uF, Capacitor_SMD:C_0402_1005Metric, symbol Device:C
- removed J1: Conn_01x04, zhangxiaofei:SWD, symbol Connector_Generic:Conn_01x04
- removed J2: USB_A, zhangxiaofei:mini_usb, symbol Connector:USB_A
- removed U1: nRF52840, Package_DFN_QFN:Nordic_AQFN-73-1EP_7x7mm_P0.5mm, symbol NRF52840-rescue:nRF52840-MCU_Nordic
- removed Y1: 32M, Crystal:Crystal_SMD_2016-4Pin_2.0x1.6mm, symbol Device:Crystal_GND24
- added L2: 10uH, Inductor_SMD:L_0603_1608Metric_Pad1.05x0.95mm_HandSolder, symbol Device:L
- added L3: 15nH, Inductor_SMD:L_0402_1005Metric, symbol Device:L
- added U1: nRF52832-QFxx, Package_DFN_QFN:QFN-48-1EP_6x6mm_P0.4mm_EP4.6x4.6mm, symbol NRF52840-rescue:nRF52832-QFxx
- added X1: 32mHz, Crystal:Crystal_SMD_2016-4Pin_2.0x1.6mm, symbol Device:Crystal_GND24_Small
- added X2: 32.768kHz, Crystal:Crystal_SMD_3215-2Pin_3.2x1.5mm, symbol Device:Crystal
- AE1: footprint RF_spark:TRACE_ANTENNA_2.4GHZ_25.7MM -> RF_Antenna:Texas_SWRA117D_2.4GHz_Right
- C1, C2, C3, C8: footprint Capacitor_SMD:C_0201_0603Metric -> Capacitor_SMD:C_0402_1005Metric
- C10: value NC -> 1uF; footprint Capacitor_SMD:C_0201_0603Metric -> Capacitor_SMD:C_0603_1608Metric_Pad1.05x0.95mm_HandSolder
- C11: value 100pF -> 12pF; footprint Capacitor_SMD:C_0201_0603Metric -> Capacitor_SMD:C_0402_1005Metric
- C12: value 100nF -> 12pF; footprint Capacitor_SMD:C_0201_0603Metric -> Capacitor_SMD:C_0402_1005Metric
- C4: value 0.5pF -> 100nF; footprint Capacitor_SMD:C_0201_0603Metric -> Capacitor_SMD:C_0402_1005Metric
- C5: value 100nf -> 100nF; footprint Capacitor_SMD:C_0201_0603Metric -> Capacitor_SMD:C_0402_1005Metric
- C6: value 4.7uF -> NC
- C7: value 100nF -> 100pF; footprint Capacitor_SMD:C_0201_0603Metric -> Capacitor_SMD:C_0402_1005Metric
- C9: value 820pF -> 100nF; footprint Capacitor_SMD:C_0402_1005Metric -> Capacitor_SMD:C_0603_1608Metric_Pad1.05x0.95mm_HandSolder
- L1: value 4.7nH -> 3.9nH; footprint Inductor_SMD:L_0201_0603Metric -> Inductor_SMD:L_0402_1005Metric
Connections:
- net +3V3: now also C5.1, C9.1, U1.13 (VDD), U1.36 (VDD), U1.48 (VDD); no longer C12.1, C6.1, C7.1
- net GND: now also C10.2, C11.2, C6.1, C7.1, U1.31 (VSS), U1.45 (VSS), U1.49 (VSS), X1.2, X1.4; no longer C10.1, C11.1, C6.2, C7.2
- net at C2.2: now also U1.35 (XC2), X1.1
- net at C1.2: now also U1.34 (XC1), X1.3
- net at C3.2, L1.2: now also U1.30 (ANT)
- net at AE1.1 (A), L1.1: no longer C4.1
- new net: C4.1, U1.1 (DEC1)
- new net: C11.1, U1.2 (P0.00/XL1), X2.1
- new net: C12.1, U1.3 (P0.01/XL2), X2.2
- new net: C6.2, U1.32 (DEC2)
- new net: C7.2, U1.33 (DEC3)
- new net: C10.1, L3.1, U1.46 (DEC4)
- new net: L2.2, U1.47 (DCC)
- new net: L2.1, L3.2
- no-connect marks 51 -> 33

Commit message: ...
Parts:
- removed AE1: Antenna, RF_Antenna:Texas_SWRA117D_2.4GHz_Right, symbol Device:Antenna
- added AE1: Antenna_Dipole, RF_Antenna:Texas_SWRA117D_2.4GHz_Left, symbol Device:Antenna_Dipole
- added C13: 0.5pF, Capacitor_SMD:C_0402_1005Metric, symbol Device:C
- added J1, J2: Conn_01x14, zhangxiaofei:half_hole_1, symbol Connector_Generic:Conn_01x14
- added J3: Conn_01x12, zhangxiaofei:half_hole_12, symbol Connector_Generic:Conn_01x12
- added J4, J5: Conn_01x02, zhangxiaofei:half_hole_2, symbol Connector_Generic:Conn_01x02
Connections:
- net +3V3: now also J2.1 (Pin_1), J2.12 (Pin_12), J3.4 (Pin_4)
- net GND: now also AE1.2, C13.1, J1.1 (Pin_1), J2.10 (Pin_10), J2.11 (Pin_11), J2.13 (Pin_13), J2.9 (Pin_9), J4.1 (Pin_1), J4.2 (Pin_2), J5.1 (Pin_1), J5.2 (Pin_2)
- net P0.8: now reaches U1.10 (P0.08)
- net P0.8: now also J3.7 (Pin_7)
- net P0.9: now reaches U1.11 (NFC1/P0.09)
- net P0.9: now also J3.6 (Pin_6)
- net P0.10: now reaches U1.12 (NFC2/P0.10)
- net P0.10: now also J3.5 (Pin_5)
- net P0.11: now reaches U1.14 (P0.11)
- net P0.11: now also J3.3 (Pin_3)
- net P0.12: now reaches U1.15 (P0.12)
- net P0.12: now also J3.2 (Pin_2)
- net P0.13: now reaches U1.16 (P0.13)
- net P0.13: now also J3.1 (Pin_1)
- net P0.14: now reaches U1.17 (P0.14)
- net P0.14: now also J1.14 (Pin_14)
- net P0.15: now reaches U1.18 (P0.15)
- net P0.15: now also J1.13 (Pin_13)
- net P0.16: now reaches U1.19 (P0.16)
- net P0.16: now also J1.12 (Pin_12)
- net P0.17: now reaches U1.20 (P0.17)
- net P0.17: now also J1.11 (Pin_11)
- net P0.18: now reaches U1.21 (P0.18/SWO)
- net P0.18: now also J1.10 (Pin_10)
- net P0.19: now reaches U1.22 (P0.19)
- net P0.19: now also J1.9 (Pin_9)
- net P0.20: now reaches U1.23 (P0.20)
- net P0.20: now also J1.8 (Pin_8)
- net P0.21: now reaches U1.24 (P0.21/~RESET)
- net P0.21: now also J1.7 (Pin_7)
- net SWDCLK: now reaches U1.25 (SWDCLK)
- net SWDCLK: now also J1.6 (Pin_6)
- net SWDIO: now reaches U1.26 (SWDIO)
- net SWDIO: now also J1.5 (Pin_5)
- net P0.22: now reaches U1.27 (P0.22)
- net P0.22: now also J1.4 (Pin_4)
- net P0.23: now reaches U1.28 (P0.23)
- net P0.23: now also J1.3 (Pin_3)
- net P0.24: now reaches U1.29 (P0.24)
- net P0.24: now also J1.2 (Pin_2)
- net P0.25: now reaches U1.37 (P0.25)
- net P0.25: now also J2.2 (Pin_2)
- net P0.26: now reaches U1.38 (P0.26)
- net P0.26: now also J2.3 (Pin_3)
- net P0.27: now reaches U1.39 (P0.27)
- net P0.27: now also J2.4 (Pin_4)
- net P0.2: now reaches U1.4 (P0.02/AIN0)
- net P0.2: now also J2.14 (Pin_14)
- net P0.28: now reaches U1.40 (P0.28/AIN4)
- net P0.28: now also J2.5 (Pin_5)
- net P0.29: now reaches U1.41 (P0.29/AIN5)
- net P0.29: now also J2.6 (Pin_6)
- net P0.30: now reaches U1.42 (P0.30/AIN6)
- net P0.30: now also J2.7 (Pin_7)
- net P0.31: now reaches U1.43 (P0.31/AIN7)
- net P0.31: now also J2.8 (Pin_8)
- net P0.3: now reaches U1.5 (P0.03/AIN1)
- net P0.3: now also J3.12 (Pin_12)
- net P0.4: now reaches U1.6 (P0.04/AIN2)
- net P0.4: now also J3.11 (Pin_11)
- net P0.5: now reaches U1.7 (P0.05/AIN3)
- net P0.5: now also J3.10 (Pin_10)
- net P0.6: now reaches U1.8 (P0.06)
- net P0.6: now also J3.9 (Pin_9)
- net P0.7: now reaches U1.9 (P0.07)
- net P0.7: now also J3.8 (Pin_8)
- net at L1.1: now also AE1.1, C13.2
- no-connect marks 33 -> 1
Other:
- moved on the sheet: C8
