File: NRF52840.sch (KiCad schematic (older format))
At the start: 27 parts, among them J1 Conn_01x04, J2 USB_A, U1 nRF52840, Y1 32M

Commit message: ...
Parts:
- removed C10, C13, C25: NC, Capacitor_SMD:C_0402_1005Metric, symbol Device:C
- AE1: footprint RF_spark:TRACE_ANTENNA_2.4GHZ_25.7MM -> zhangxiaofei:2.4g_ANTENNA
- J1: footprint zhangxiaofei:SWD -> Connector_PinHeader_2.54mm:PinHeader_1x04_P2.54mm_Vertical
- J2: footprint zhangxiaofei:USB_PCB -> Connector_USB:USB_A_CNCTech_1001-011-01101_Horizontal; symbol Connector:USB_A -> NRF52840-rescue:USB_A-Connector
- U1: footprint Package_DFN_QFN:Nordic_AQFN-73-1EP_7x7mm_P0.5mm -> zhangxiaofei:Nordic_AQFN-73-1EP_7x7mm_P0.5mm; symbol MCU_Nordic:nRF52840 -> NRF52840-rescue:nRF52840-MCU_Nordic
Connections:
- net GND: now also J2.5 (Shield)
Changed lines of the file:
@@
-$EndComp
-$Comp
-L Device:C C25
-U 1 1 5F20DA14
-P 16600 8050
-F 0 "C25" H 16715 8096 50  0000 L CNN
-F 1 "NC" H 16715 8005 50  0000 L CNN
-F 2 "Capacitor_SMD:C_0402_1005Metric" H 16638 7900 50  0001 C CNN
-F 3 "~" H 16600 8050 50  0001 C CNN
-	1    16600 8050
-	1    0    0    -1
 $EndComp
 $Comp
@@
 Wire Wire Line
 	15800 7900 16100 7900
-Wire Wire Line
-	16100 7900 16600 7900
 Connection ~ 16100 7900
-Connection ~ 16600 7900
-Wire Wire Line
-	16600 7900 16950 7900
 Wire Wire Line
 	17250 7900 17500 7900
@@
 Wire Wire Line
 	16100 8450 16600 8450
-Wire Wire Line
-	16600 8200 16600 8450
 Connection ~ 16600 8450
 Wire Wire Line
@@
 $EndComp
 $Comp
-L MCU_Nordic:nRF52840 U1
+L NRF52840-rescue:nRF52840-MCU_Nordic U1
 U 1 1 5F1F0A1E
 P 12150 7800
 F 0 "U1" H 12150 9681 50  0000 C CNN
-F 1 "nRF52840" H 12150 9590 50  0000 C CNN
-F 2 "Package_DFN_QFN:Nordic_AQFN-73-1EP_7x7mm_P0.5mm" H 12300 3100 50  0001 C CNN
+F 1 "nRF52840" H 12100 7850 50  0000 C CNN
+F 2 "zhangxiaofei:Nordic_AQFN-73-1EP_7x7mm_P0.5mm" H 12300 3100 50  0001 C CNN
 F 3 "http://infocenter.nordicsemi.com/topic/com.nordic.infocenter.nrf52/dita/nrf52/chips/nrf52840.html" H 11900 9700 50  0001 C CNN
 	1    12150 7800
@@
 Wire Wire Line
 	13850 7700 15700 7700
-Wire Wire Line
-	15700 7700 15700 7400
 $Comp
 L Device:C C11
@@
 	0    1    1    0
 $EndComp
-$Comp
-L Device:C C10
-U 1 1 5F222ABB
-P 16150 7400
-F 0 "C10" V 15898 7400 50  0000 C CNN
-F 1 "NC" V 15989 7400 50  0000 C CNN
-F 2 "Capacitor_SMD:C_0402_1005Metric" H 16188 7250 50  0001 C CNN
-F 3 "~" H 16150 7400 50  0001 C CNN
-	1    16150 7400
-	0    1    1    0
-$EndComp
-Wire Wire Line
-	15700 7400 16000 7400
-Connection ~ 15700 7400
-Wire Wire Line
-	16300 7400 16450 7400
-Wire Wire Line
-	16450 7400 16450 7600
 Wire Wire Line
 	16300 6850 16450 6850
-Wire Wire Line
-	16450 6850 16450 7400
-Connection ~ 16450 7400
 Wire Wire Line
 	15550 6850 16000 6850
@@
 $EndComp
 Wire Wire Line
-	15700 3600 15700 7400
-Wire Wire Line
 	11550 6100 11550 3600
 Wire Wire Line
@@
 $EndComp
 Wire Wire Line
-	12750 5150 12750 6100
-$Comp
-L Device:C C13
-U 1 1 5F24071E
-P 12750 5000
-F 0 "C13" H 12865 5046 50  0000 L CNN
-F 1 "NC" H 12865 4955 50  0000 L CNN
-F 2 "Capacitor_SMD:C_0402_1005Metric" H 12788 4850 50  0001 C CNN
-F 3 "~" H 12750 5000 50  0001 C CNN
-	1    12750 5000
-	1    0    0    -1
-$EndComp
-$Comp
-L power:GND #PWR019
-U 1 1 5F24136A
-P 12750 4850
-F 0 "#PWR019" H 12750 4600 50  0001 C CNN
-F 1 "GND" H 12755 4677 50  0000 C CNN
-F 2 "" H 12750 4850 50  0001 C CNN
-F 3 "" H 12750 4850 50  0001 C CNN
-	1    12750 4850
-	-1   0    0    1
-$EndComp
-Wire Wire Line
 	13050 6100 13050 5500
 Wire Wire Line
@@
 F 0 "J1" H 8680 11342 50  0000 L CNN
 F 1 "Conn_01x04" H 8680 11251 50  0000 L CNN
-F 2 "zhangxiaofei:SWD" H 8600 11350 50  0001 C CNN
+F 2 "Connector_PinHeader_2.54mm:PinHeader_1x04_P2.54mm_Vertical" H 8600 11350 50  0001 C CNN
 F 3 "~" H 8600 11350 50  0001 C CNN
 	1    8600 11350
@@
 F 0 "AE1" V 18054 8030 50  0000 L CNN
 F 1 "Antenna" V 18145 8030 50  0000 L CNN
-F 2 "RF_spark:TRACE_ANTENNA_2.4GHZ_25.7MM" H 18100 7900 50  0001 C CNN
+F 2 "zhangxiaofei:2.4g_ANTENNA" H 18100 7900 50  0001 C CNN
 F 3 "~" H 18100 7900 50  0001 C CNN
 	1    18100 7900
@@
 NoConn ~ 12950 6100
 $Comp
-L Connector:USB_A J2
+L NRF52840-rescue:USB_A-Connector J2
 U 1 1 5F292A35
 P 9900 11450
 F 0 "J2" H 9957 11917 50  0000 C CNN
 F 1 "USB_A" H 9957 11826 50  0000 C CNN
-F 2 "zhangxiaofei:USB_PCB" H 10050 11400 50  0001 C CNN
+F 2 "Connector_USB:USB_A_CNCTech_1001-011-01101_Horizontal" H 10050 11400 50  0001 C CNN
 F 3 " ~" H 10050 11400 50  0001 C CNN
 	1    9900 11450
@@
 	1    0    0    -1
 $EndComp
-NoConn ~ 9800 11850
+Wire Wire Line
+	16100 7900 16950 7900
+Wire Wire Line
+	15700 3600 15700 7700
+Wire Wire Line
+	16450 6850 16450 7600
+NoConn ~ 12750 6100
+Wire Wire Line
+	9800 11850 9800 12050
+Wire Wire Line
+	9800 12050 9850 12050
+Connection ~ 9850 12050
 $EndSCHEMATC
