File: NRF52840.kicad_pcb (KiCad board)
At the start: 2 copper layers, 31.2 x 11.3 mm, 26 parts, among them J1 Conn_01x04, J2 USB_A, U1 nRF52840, Y1 32M

Commit message: ...
Parts:
- removed C10, C13, C25: NC, Capacitor_SMD:C_0402_1005Metric
- removed C12, C8: 100nF, Capacitor_SMD:C_0402_1005Metric
- removed C14: 1.0uF, Capacitor_SMD:C_0603_1608Metric
- removed C19, C6: 4.7uF, Capacitor_SMD:C_0603_1608Metric
- removed C26: 1.5pF, Capacitor_SMD:C_0402_1005Metric
- removed C7: 100nf, Capacitor_SMD:C_0402_1005Metric
- removed R1: 0R, Capacitor_SMD:C_0402_1005Metric
- C11, C15, C16, C20, C3, C4, C5, C9, L1, U1: moved to B.Cu
- J1: value Conn_01x04 -> Conn_01x02; footprint zhangxiaofei:SWD -> zhangxiaofei:SWD_2_PIN
- J2: moved to F.Cu
- moved C15 48.8 mm to (134.8, 156.9)
- moved C5 43.8 mm to (123.6, 157.4)
- moved C2 43.1 mm to (129.4, 158.5), turned to 180 degrees
- moved C11 41.5 mm to (134.3, 158.2)
- moved J2 40.5 mm to (124.4, 154.7), turned to 90 degrees
- moved Y1 39.9 mm to (129.6, 156.7)
- moved L1 39.3 mm to (135.2, 155.6)
- moved C4 39.2 mm to (136.6, 155.1)
- moved C3 38.7 mm to (133.8, 155.1), turned to 270 degrees
- moved U1 38.1 mm to (128.7, 155.2)
- moved C1 37.5 mm to (129.9, 154.8), turned to 0 degrees
- moved C16 37.4 mm to (122.9, 154.4)
- moved C20 37.0 mm to (123.0, 152.3)
- moved C9 36.3 mm to (134.3, 153.7), turned to 0 degrees
- moved J1 34.1 mm to (134.3, 151.4), turned to 180 degrees
Connections:
- U1 pad A10: Net-(U1-PadA10) -> (no net)
- U1 pad A12: Net-(U1-PadA12) -> (no net)
- U1 pad A14: Net-(U1-PadA14) -> (no net)
- U1 pad A16: Net-(U1-PadA16) -> (no net)
- U1 pad A18: Net-(C13-Pad2) -> (no net)
- U1 pad A20: Net-(U1-PadA20) -> (no net)
- U1 pad A22: +3V3 -> (no net)
- U1 pad A8: Net-(U1-PadA8) -> (no net)
- U1 pad AB2: Net-(U1-PadAB2) -> (no net)
- U1 pad AC11: Net-(U1-PadAC11) -> (no net)
- U1 pad AC13: Net-(U1-PadAC13) -> (no net)
- U1 pad AC15: Net-(U1-PadAC15) -> (no net)
- U1 pad AC17: Net-(U1-PadAC17) -> (no net)
- U1 pad AC19: Net-(U1-PadAC19) -> (no net)
- U1 pad AC21: Net-(U1-PadAC21) -> (no net)
- U1 pad AC9: Net-(U1-PadAC9) -> (no net)
- U1 pad AD10: Net-(U1-PadAD10) -> (no net)
- U1 pad AD12: Net-(U1-PadAD12) -> (no net)
- U1 pad AD14: +3V3 -> (no net)
- U1 pad AD16: Net-(U1-PadAD16) -> (no net)
- U1 pad AD18: Net-(U1-PadAD18) -> (no net)
- U1 pad AD20: Net-(U1-PadAD20) -> (no net)
- U1 pad AD22: Net-(U1-PadAD22) -> (no net)
- U1 pad AD23: +3V3 -> (no net)
- U1 pad AD8: Net-(U1-PadAD8) -> (no net)
- U1 pad B1: +3V3 -> (no net)
- U1 pad B11: Net-(U1-PadB11) -> (no net)
- U1 pad B13: Net-(U1-PadB13) -> (no net)
- U1 pad B15: Net-(U1-PadB15) -> (no net)
- U1 pad B17: Net-(U1-PadB17) -> (no net)
- U1 pad B19: Net-(U1-PadB19) -> (no net)
- U1 pad B3: Net-(U1-PadB3) -> (no net)
- U1 pad B9: Net-(U1-PadB9) -> (no net)
- U1 pad D2: Net-(U1-PadD2) -> (no net)
- U1 pad F2: Net-(U1-PadF2) -> (no net)
- U1 pad G1: Net-(U1-PadG1) -> (no net)
- U1 pad H2: Net-(U1-PadH2) -> (no net)
- U1 pad J1: Net-(U1-PadJ1) -> (no net)
- U1 pad J24: Net-(U1-PadJ24) -> (no net)
- U1 pad K2: Net-(U1-PadK2) -> (no net)
- U1 pad L1: Net-(U1-PadL1) -> (no net)
- U1 pad L24: Net-(U1-PadL24) -> (no net)
- U1 pad M2: Net-(U1-PadM2) -> (no net)
- U1 pad N1: Net-(U1-PadN1) -> (no net)
- U1 pad P2: Net-(U1-PadP2) -> (no net)
- U1 pad P23: Net-(U1-PadP23) -> (no net)
- U1 pad R1: Net-(U1-PadR1) -> (no net)
- U1 pad R24: Net-(U1-PadR24) -> (no net)
- U1 pad T2: Net-(U1-PadT2) -> (no net)
- U1 pad T23: Net-(U1-PadT23) -> (no net)
- U1 pad U1: Net-(U1-PadU1) -> (no net)
- U1 pad U24: Net-(U1-PadU24) -> (no net)
- U1 pad V23: Net-(U1-PadV23) -> (no net)
- U1 pad W1: +3V3 -> (no net)
- U1 pad W24: Net-(U1-PadW24) -> (no net)
- U1 pad Y23: Net-(U1-PadY23) -> (no net)
Routing:
- net +3V3: track 42.5 -> 0.00 mm, vias 5 -> 0
- net Net-(AE1-Pad1) (its old number): track 29.8 -> 0.00 mm
- net +5V: track 35.3 -> 13.8 mm
- net GND: track 79.6 -> 67.5 mm, vias 30 -> 5
- net Net-(AE1-Pad1): track 7.90 -> 19.6 mm
- net SWDIO: track 10.4 -> 1.88 mm, vias 1 -> 0
- net SWDCLK: track 10.7 -> 4.30 mm, vias 1 -> 0
- net D+: track 6.31 -> 10.8 mm
- net Net-(C20-Pad1): track 6.00 -> 3.00 mm
- net D-: track 17.8 -> 15.0 mm
- net Net-(C5-Pad1): track 3.95 -> 1.45 mm
- net Net-(C13-Pad2): track 1.85 -> 0.00 mm
- net Net-(C1-Pad2): track 7.76 -> 6.09 mm, vias 0 -> 1
- net Net-(C2-Pad2): track 3.94 -> 5.51 mm, vias 0 -> 1
- net Net-(C15-Pad1): track 16.5 -> 17.8 mm, vias 2 -> 0
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Other:
- board size 31.2 x 11.3 mm -> 20 x 9.6 mm
- board text added: "c"
- board text added: "i"
- board text removed: "3V3"
- board text removed: "5"
- board text removed: "D+"
- board text removed: "D-"
- board text removed: "GND"
- board text removed: "SWDCLK"
- board text removed: "SWDIO"

Commit message: ...
Parts:
- removed C16: 4.7uF, Capacitor_SMD:C_0603_1608Metric
- added 2.4: 2.4g_taocitianxian, zhangxiaofei:2.4g_taocitianxian, F.Cu at (138.8, 154.7)
- added C10: NC, Capacitor_SMD:C_0201_0603Metric, F.Cu at (133.0, 153.6)
- added C12: 100nF, Capacitor_SMD:C_0201_0603Metric, F.Cu at (128.2, 150.8)
- added C13: NC, Capacitor_SMD:C_0201_0603Metric, F.Cu at (126.7, 150.8)
- added C14: 1.0uf, Capacitor_SMD:C_0402_1005Metric, F.Cu at (122.2, 152.3)
- added C19: 4.7uF, Capacitor_SMD:C_0402_1005Metric, F.Cu at (122.2, 158.8)
- added C6: 4.7uF, Capacitor_SMD:C_0402_1005Metric, F.Cu at (122.2, 156.3)
- added C7: 100nF, Capacitor_SMD:C_0201_0603Metric, F.Cu at (126.9, 159.4)
- added C8: 100nF, Capacitor_SMD:C_0201_0603Metric, F.Cu at (129.5, 159.4)
- C1, C2: footprint Capacitor_SMD:C_0402_1005Metric -> Capacitor_SMD:C_0201_0603Metric
- C11, C5: footprint Capacitor_SMD:C_0402_1005Metric -> Capacitor_SMD:C_0201_0603Metric; moved to F.Cu
- C15, C20: footprint Capacitor_SMD:C_0603_1608Metric -> Capacitor_SMD:C_0402_1005Metric; moved to F.Cu
- C3: value 1.0pF -> 0.8pF; footprint Capacitor_SMD:C_0402_1005Metric -> Capacitor_SMD:C_0201_0603Metric; moved to F.Cu
- C4: value 1.0pF -> 0.5pF; footprint Capacitor_SMD:C_0402_1005Metric -> Capacitor_SMD:C_0201_0603Metric; moved to F.Cu
- C9, U1: moved to F.Cu
- J1: value Conn_01x02 -> Conn_01x04; footprint zhangxiaofei:SWD_2_PIN -> zhangxiaofei:SWD
- J2: footprint zhangxiaofei:USB_PCB -> zhangxiaofei:mini_usb; moved to B.Cu
- L1: value 3.9nH -> 4.7nH; footprint Inductor_SMD:L_0402_1005Metric -> Inductor_SMD:L_0201_0603Metric; moved to F.Cu
- moved C15 11.7 mm to (124.9, 150.7)
- moved C2 10.2 mm to (136.4, 151.0)
- moved Y1 6.65 mm to (134.2, 151.8), turned to 180 degrees
- moved C11 6.16 mm to (131.8, 152.6)
- moved C20 5.64 mm to (122.2, 157.9)
- moved C9 4.53 mm to (131.5, 157.3), turned to 270 degrees
- moved J1 4.33 mm to (131.4, 154.6), turned to 270 degrees
- moved C1 3.94 mm to (131.8, 151.3)
- moved C5 3.78 mm to (122.2, 153.9)
- moved C4 3.11 mm to (133.5, 154.8), turned to 270 degrees
- moved L1 3.08 mm to (132.4, 154.4)
- moved C3 2.61 mm to (131.2, 154.8), turned to 90 degrees
- moved U1 1.75 mm to (127.0, 155.0)
- moved J2 0.79 mm to (124.3, 155.5), turned to 270 degrees
Connections:
- J1 pad 1: SWDCLK -> GND
- J1 pad 2: SWDIO -> SWDCLK
- U1 pad A18: (no net) -> Net-(C13-Pad1)
- U1 pad A22: (no net) -> +3V3
- U1 pad AD14: (no net) -> +3V3
- U1 pad AD23: (no net) -> +3V3
- U1 pad B1: (no net) -> +3V3
- U1 pad W1: (no net) -> +3V3
Routing:
- net GND: track 67.5 -> 36.4 mm, vias 5 -> 40
- net +3V3: track 0.00 -> 13.3 mm, vias 0 -> 5
- net Net-(AE1-Pad1): track 19.6 -> 8.92 mm
- net +5V: track 13.8 -> 19.9 mm, vias 1 -> 2
- net SWDCLK: track 4.30 -> 9.78 mm, vias 0 -> 1
- net SWDIO: track 1.88 -> 7.14 mm, vias 0 -> 1
- net D-: track 15.0 -> 12.4 mm, vias 1 -> 2
- net Net-(C2-Pad2): track 5.51 -> 7.47 mm, vias 1 -> 0
- net Net-(C1-Pad2): track 6.09 -> 4.16 mm, vias 1 -> 0
- net Net-(C13-Pad1): track 0.00 -> 1.64 mm
- net Net-(C10-Pad2): track 17.8 -> 19.4 mm, vias 0 -> 2
- net Net-(C3-Pad2): track 3.70 -> 2.61 mm
- net Net-(C11-Pad2): track 2.94 -> 1.87 mm
- net Net-(C20-Pad1): track 3.00 -> 2.37 mm
- net Net-(C9-Pad1): track 2.59 -> 2.07 mm
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- added copper zone on VCC2.Cu, net +3V3
- added copper zone on GND1.Cu, net GND
Other:
- outline, holes or cut-outs redrawn
- copper layers 2 -> 4
- rule via_min_drill: 0.3 -> 0.2
- rule via_min_size: 0.4 -> 0.2
- board text added: "3.3"
- board text added: "CLK"
- board text added: "GND"
- board text added: "IO"
- board text removed: "c"
- board text removed: "i"

Commit message: ...
Parts:
- removed 2.4: 2.4g_taocitianxian, zhangxiaofei:2.4g_taocitianxian
- removed C13: NC, Capacitor_SMD:C_0201_0603Metric
- removed C14: 1.0uf, Capacitor_SMD:C_0402_1005Metric
- removed C15: 1.0uF, Capacitor_SMD:C_0402_1005Metric
- removed C19, C20: 4.7uF, Capacitor_SMD:C_0402_1005Metric
- removed J1: Conn_01x04, zhangxiaofei:SWD
- removed J2: USB_A, zhangxiaofei:mini_usb
- removed Y1: 32M, Crystal:Crystal_SMD_2016-4Pin_2.0x1.6mm
- added AE1: Antenna, RF_Antenna:Texas_SWRA117D_2.4GHz_Right, F.Cu at (117.8, 143.2)
- added L2: 10uH, Inductor_SMD:L_0603_1608Metric_Pad1.05x0.95mm_HandSolder, F.Cu at (124.9, 145.7)
- added L3: 15nH, Inductor_SMD:L_0402_1005Metric, F.Cu at (119.1, 151.1)
- added X1: 32mHz, Crystal:Crystal_SMD_2016-4Pin_2.0x1.6mm, F.Cu at (124.7, 148.8)
- added X2: 32.768kHz, Crystal:Crystal_SMD_3215-2Pin_3.2x1.5mm, F.Cu at (115.9, 146.2)
- C1, C2, C3, C8: footprint Capacitor_SMD:C_0201_0603Metric -> Capacitor_SMD:C_0402_1005Metric
- C10: value NC -> 1uF; footprint Capacitor_SMD:C_0201_0603Metric -> Capacitor_SMD:C_0603_1608Metric_Pad1.05x0.95mm_HandSolder
- C11: value 100pF -> 12pF; footprint Capacitor_SMD:C_0201_0603Metric -> Capacitor_SMD:C_0402_1005Metric
- C12: value 100nF -> 12pF; footprint Capacitor_SMD:C_0201_0603Metric -> Capacitor_SMD:C_0402_1005Metric
- C4: value 0.5pF -> 100nF; footprint Capacitor_SMD:C_0201_0603Metric -> Capacitor_SMD:C_0402_1005Metric
- C5: value 100nf -> 100nF; footprint Capacitor_SMD:C_0201_0603Metric -> Capacitor_SMD:C_0402_1005Metric
- C6: value 4.7uF -> NC
- C7: value 100nF -> 100pF; footprint Capacitor_SMD:C_0201_0603Metric -> Capacitor_SMD:C_0402_1005Metric
- C9: value 820pF -> 100nF; footprint Capacitor_SMD:C_0402_1005Metric -> Capacitor_SMD:C_0603_1608Metric_Pad1.05x0.95mm_HandSolder
- L1: value 4.7nH -> 3.9nH; footprint Inductor_SMD:L_0201_0603Metric -> Inductor_SMD:L_0402_1005Metric
- U1: value nRF52840 -> nRF52832-QFxx; footprint Package_DFN_QFN:Nordic_AQFN-73-1EP_7x7mm_P0.5mm -> Package_DFN_QFN:QFN-48-1EP_6x6mm_P0.4mm_EP4.6x4.6mm
- moved C9 18.0 mm to (115.5, 149.1), turned to 0 degrees
- moved U1 15.3 mm to (134.1, 141.5)
- moved C6 15.2 mm to (133.9, 146.6), turned to 0 degrees
- moved C10 14.2 mm to (120.6, 146.9), turned to 0 degrees
- moved C11 13.1 mm to (119.1, 149.1), turned to 0 degrees
- moved C8 12.9 mm to (131.0, 146.6)
- moved C7 11.5 mm to (131.0, 148.6), turned to 0 degrees
- moved C3 9.85 mm to (136.8, 146.6), turned to 0 degrees
- moved C5 9.37 mm to (131.0, 150.6), turned to 0 degrees
- moved L1 7.78 mm to (128.0, 148.0), turned to 0 degrees
- moved C4 6.21 mm to (133.9, 148.6), turned to 0 degrees
- moved C1 5.67 mm to (136.8, 148.6)
- moved C2 2.55 mm to (133.9, 150.6), turned to 0 degrees
- moved C12 0.82 mm to (128.0, 150.0), turned to 0 degrees
Connections:
- C10 pad 1: GND -> Net-(C10-Pad1)
- C10 pad 2: Net-(C10-Pad2) -> GND
- C11 pad 1: GND -> Net-(C11-Pad1)
- C11 pad 2: Net-(C11-Pad2) -> GND
- C12 pad 1: +3V3 -> Net-(C12-Pad1)
- C4 pad 1: Net-(AE1-Pad1) -> Net-(C4-Pad1)
- C5 pad 1: Net-(C5-Pad1) -> +3V3
- C6 pad 1: +3V3 -> GND
- C6 pad 2: GND -> Net-(C6-Pad2)
- C7 pad 1: +3V3 -> GND
- C7 pad 2: GND -> Net-(C7-Pad2)
- C9 pad 1: Net-(C9-Pad1) -> +3V3
Routing:
- net GND: track 36.4 -> 0.00 mm, vias 40 -> 0
- net +5V: track 19.9 -> 0.00 mm, vias 2 -> 0
- net Net-(C10-Pad2): track 19.4 -> 0.00 mm, vias 2 -> 0
- net +3V3: track 13.3 -> 0.00 mm, vias 5 -> 0
- net D-: track 12.4 -> 0.00 mm, vias 2 -> 0
- net D+: track 11.3 -> 0.00 mm, vias 2 -> 0
- net SWDCLK: track 9.78 -> 0.00 mm, vias 1 -> 0
- net Net-(AE1-Pad1): track 8.92 -> 0.00 mm
- net Net-(C2-Pad2): track 7.47 -> 0.00 mm
- net SWDIO: track 7.14 -> 0.00 mm, vias 1 -> 0
- net Net-(C1-Pad2): track 4.16 -> 0.00 mm
- net Net-(C3-Pad2): track 2.61 -> 0.00 mm
- net Net-(C20-Pad1): track 2.37 -> 0.00 mm
- net Net-(C9-Pad1): track 2.07 -> 0.00 mm
- net Net-(C11-Pad2): track 1.87 -> 0.00 mm
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- removed copper zone on VCC2.Cu, net +3V3
- removed copper zone on B.Cu, net GND
- removed copper zone on F.Cu, net GND
- removed copper zone on GND1.Cu, net GND
Other:
- board outline removed
- board text removed: "3.3"
- board text removed: "CLK"
- board text removed: "GND"
- board text removed: "IO"

Commit message: ...
Parts:
- added C13: 0.5pF, Capacitor_SMD:C_0402_1005Metric, F.Cu at (135.1, 122.1)
- added J1: Conn_01x14, zhangxiaofei:half_hole_1, F.Cu at (124.8, 129.4)
- added J2: Conn_01x14, zhangxiaofei:half_hole_1, F.Cu at (124.8, 112.1)
- added J3: Conn_01x12, zhangxiaofei:half_hole_12, F.Cu at (115.5, 121.3)
- added J4: Conn_01x02, zhangxiaofei:half_hole_2, F.Cu at (136.9, 129.5)
- added J5: Conn_01x02, zhangxiaofei:half_hole_2, F.Cu at (136.9, 112.0)
- AE1: value Antenna -> Antenna_Dipole; footprint RF_Antenna:Texas_SWRA117D_2.4GHz_Right -> RF_Antenna:Texas_SWRA117D_2.4GHz_Left
- moved L3 37.1 mm to (124.4, 114.4), turned to 90 degrees
- moved C2 34.8 mm to (131.5, 115.8), turned to 270 degrees
- moved X1 34.0 mm to (133.5, 115.9)
- moved C4 33.5 mm to (121.9, 117.4), turned to 180 degrees
- moved C9 33.4 mm to (120.2, 116.1), turned to 180 degrees
- moved C1 32.8 mm to (135.6, 115.8), turned to 90 degrees
- moved C10 31.8 mm to (123.1, 115.1), turned to 270 degrees
- moved C8 30.8 mm to (130.5, 115.8), turned to 90 degrees
- moved L2 30.6 mm to (125.7, 115.1), turned to 270 degrees
- moved C11 30.4 mm to (121.5, 118.8), turned to 270 degrees
- moved C12 29.8 mm to (119.9, 121.4), turned to 180 degrees
- moved C7 29.2 mm to (132.7, 119.5), turned to 180 degrees
- moved X2 27.6 mm to (119.8, 118.9), turned to 90 degrees
- moved AE1 27.3 mm to (138.3, 125.2), turned to 270 degrees
- moved C5 26.9 mm to (122.2, 125.1), turned to 90 degrees
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Connections:
- AE1 pad 2: (no net) -> GND
- U1 pad 10: (no net) -> P0.8
- U1 pad 11: (no net) -> P0.9
- U1 pad 12: (no net) -> P0.10
- U1 pad 14: (no net) -> P0.11
- U1 pad 15: (no net) -> P0.12
- U1 pad 16: (no net) -> P0.13
- U1 pad 17: (no net) -> P0.14
- U1 pad 18: (no net) -> P0.15
- U1 pad 19: (no net) -> P0.16
- U1 pad 20: (no net) -> P0.17
- U1 pad 21: (no net) -> P0.18
- U1 pad 22: (no net) -> P0.19
- U1 pad 23: (no net) -> P0.20
- U1 pad 24: (no net) -> P0.21
- U1 pad 25: (no net) -> SWDCLK
- U1 pad 26: (no net) -> SWDIO
- U1 pad 27: (no net) -> P0.22
- U1 pad 28: (no net) -> P0.23
- U1 pad 29: (no net) -> P0.24
- U1 pad 37: (no net) -> P0.25
- U1 pad 38: (no net) -> P0.26
- U1 pad 39: (no net) -> P0.27
- U1 pad 4: (no net) -> P0.2
- U1 pad 40: (no net) -> P0.28
- U1 pad 41: (no net) -> P0.29
- U1 pad 42: (no net) -> P0.30
- U1 pad 43: (no net) -> P0.31
- U1 pad 5: (no net) -> P0.3
- U1 pad 6: (no net) -> P0.4
- U1 pad 7: (no net) -> P0.5
- U1 pad 8: (no net) -> P0.6
- U1 pad 9: (no net) -> P0.7
Routing:
- net GND: track 0.00 -> 51.4 mm, vias 0 -> 53
- net +3V3: track 0.00 -> 49.1 mm, vias 0 -> 3
- net P0.2: track 0.00 -> 16.8 mm
- net P0.3: track 0.00 -> 16.3 mm
- net P0.4: track 0.00 -> 15.4 mm
- net P0.5: track 0.00 -> 14.4 mm
- net P0.6: track 0.00 -> 13.5 mm
- net P0.7: track 0.00 -> 12.5 mm
- net Net-(C1-Pad2): track 0.00 -> 11.9 mm
- net P0.13: track 0.00 -> 11.9 mm
- net P0.12: track 0.00 -> 11.9 mm
- net P0.14: track 0.00 -> 11.7 mm
- net P0.8: track 0.00 -> 11.5 mm
- net P0.11: track 0.00 -> 11.0 mm
- net P0.15: track 0.00 -> 11.0 mm
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- added copper zone on B.Cu, net GND
- added copper zone on F.Cu, net GND
Other:
- board outline added: 28.7 x 17.5 mm
- copper layers 4 -> 2
- board text added: "3.3V"
- board text added: "C1"
- board text added: "C10"
- board text added: "C11"
- board text added: "C12"
- board text added: "C13"
- board text added: "C14"
- board text added: "C2"
- board text added: "C3"
- board text added: "C4"
- board text added: "C5"
- board text added: "C6"
- board text added: "C7"
- board text added: "C8"
- board text added: "C9"
- board text added: "GND"
- board text added: "L1"
- board text added: "L2"
- board text added: "L3"
- board text added: "P0.10"
- board text added: "P0.11"
- board text added: "P0.12"
- board text added: "P0.13"
- board text added: "P0.14"
- board text added: "P0.15"
- board text added: "P0.16"
- board text added: "P0.17"
- board text added: "P0.18"
- board text added: "P0.19"
- board text added: "P0.2"
- board text added: "P0.20"
- board text added: "P0.21"
- board text added: "P0.22"
- board text added: "P0.23"
- board text added: "P0.24"
- board text added: "P0.25"
- board text added: "P0.26"
- board text added: "P0.27"
- board text added: "P0.28"
- board text added: "P0.29"
- board text added: "P0.3"
- board text added: "P0.30"
- board text added: "P0.31"
- board text added: "P0.4"
- board text added: "P0.5"
- board text added: "P0.6"
- board text added: "P0.7"
- board text added: "P0.8"
- board text added: "P0.9"
- board text added: "SWDCLK"
- board text added: "SWDIO"
- board text added: "U1"
- board text added: "X1"
- board text added: "X2"

Commit message: ...
Routing:
- net GND: vias 53 -> 55
Other:
- board size 28.7 x 17.5 mm -> 29.7 x 19.5 mm

Commit message: ...
Routing:
- net GND: vias 55 -> 54
